File: KiCad/Bencho/carte_vitesse_1x_codincr/carte_vitesse.sch (KiCad schematic (older format))
At the start: 26 parts, among them J1 DB9, P1 VitD, P2 VitG, U1 LM324, U2 7806

Commit message: v0.9 de la carte vitesse bencho
Parts:
- removed D?: DIODESCH, symbol DIODESCH
- removed D?: BRIDGE, symbol BRIDGE
- removed GND1, GND2, GND3: Meca, symbol CONN_1
- removed HE1, HE2: HE10-10, symbol HE10-10
- removed J1: DB9, symbol DB9
- removed P1: VitD, symbol CONN_2
- removed R3, R4: 22k, symbol R
- removed R5, R6: 330, symbol R
- removed R7: 1k, symbol R
- removed R?: 6R, symbol R
- removed R?: R, symbol R
- removed U1, U? (x2): LM324, symbol LM324
- removed U2: 7806, symbol 7805
- added D2: RED, symbol LED
- added P3: GND, symbol CONN_1
- added P4: VDD, symbol CONN_1
- added P5: VCC, symbol CONN_1
- added P6: U_out, symbol CONN_1
- added P?: U_in, symbol CONN_1
- added P?: U_int, symbol CONN_1
- added P?: U_seuil, symbol CONN_1
- added RV1: 1k, symbol POT
- added RV2: 20k, symbol POT
- added U1: TL082, symbol TL082
- D1: value RED -> YELLOW
- P2: value VitG -> CAPT
- R1, R2: value 10k -> 1k
Connections:
- net labels added: U_int, U_out, capt_in
- net labels removed: +12V, +6V, +8V, -8V, -VDD, RA0, RA1, RA2, RA3, RA4, RA5, RB0, RB1, RB4, RC0, RC1, RC2, RC3, RC4, RC5, Vd, Vg, Vnd, Vng, ana, pic
- wire segments 120 -> 43
- no-connect marks 14 -> 1
Other:
- note removed: "Capteurs"
- note removed: "Carte Vitesse"
- note removed: "Connecteurs"
- note removed: "Connecteurs vers"
- note removed: "Interface"
- note removed: "Mise a l echelle 0-5V de la vitesse"
- note removed: "module de connexion"
- note removed: "témoin alim"
- moved on the sheet: C1, C2, P2
