File: KiCad/cartes_generiques/carte_std_40/carte_std_40.sch (KiCad schematic (older format))
At the start: 38 parts, among them K1 RS232, P1 ALIM, P2 CAN1, P3 CAN2, U1 7805, U2 CAN_MCP2551, U3 ICD, U4 MAX232, U5 PIC18F4580, X1 10M

Commit message: Validation cartes standard 40 & 28
Connections:
- net at U4.13 (R1IN): now also K1.1 (P1); no longer K1.2 (PM)
- net at U4.14 (T1OUT): now also K1.2 (PM); no longer K1.1 (P1)
Other:
- moved on the sheet: K1
