File: KiCad/2012_HypnoZ/carte_tdb_v0.1/carte_tdb_v0.1.sch (KiCad schematic (older format))
At the start: 5 parts

Commit message: 
Parts:
- added P?: boost_input, symbol CONN_2
- added P?: boost_analog, symbol CONN_2
- added P?: clign, symbol CONN_4
- added P?: warning, symbol CONN_2
- added R? (x5): 10k, symbol R
- added U?: TL082, symbol TL082
Connections:
- net labels added: boost_in, clign_d_in, clign_g_in, warning_in
- wire segments 13 -> 54
- no-connect marks 0 -> 1
Other:
- note added: "Boost"
- note added: "Clignotants interrupteurs"
- note added: "Freins"
- moved on the sheet: U?A

Commit message: 
Parts:
- removed R?: 10k, symbol R
- added C1: 100n, symbol C
- added C2: 100u, symbol CP
- added P10: codes, symbol CONN_2
- added P11: pleins_feux, symbol CONN_2
- added P7: clign_g, symbol CONN_2
- added P8: clign_d, symbol CONN_2
- added P9: feux_in, symbol CONN_4
- added Q1, Q2, Q3, Q4: BC237, TO92-EBC, symbol BC237
- added R1, R6, R7: 10k, symbol R
- added U? (x3): 4071, symbol 4071
- gave numbers to parts that had none: 13
Connections:
- net labels added: VCC, clign_d_out, clign_g_out, codes_in, codes_out, feux_in
- net labels removed: +5V
- wire segments 54 -> 95
- no-connect marks 1 -> 2
Other:
- note added: "Interrupteur feux"
- note added: "Logique"
- note added: "Temoins clignotant"
- note added: "Temoins feux"

Commit message: 
Parts:
- added C3, C5, C7: 100n, symbol C
- added C4, C6, C8: 100u, symbol CP
- added P12: commutateur 6pos, symbol CONN_8
- added R10, R11, R12, R13, R8, R9: 10k, symbol R
- added U3: 74LS348, symbol 74LS348
- added U4: 4049, symbol 4049
- gave numbers to parts that had none: 1
Connections:
- net labels added: comm_6pos_0, comm_6pos_1, comm_6pos_2
- wire segments 95 -> 169
- no-connect marks 2 -> 5
Other:
- note added: "Commutateur 6 positions + encodeur 3 bits"
- moved on the sheet: MEZZA2

Commit message: 
Parts:
- added P13: erreur_analog, symbol CONN_2
- added P14: erreur_1, symbol CONN_2
- added P15: erreur_2, symbol CONN_2
- added P16: erreur_3, symbol CONN_2
- added P17: cmd+, symbol CONN_2
- added Q5, Q6, Q7, Q8: BC237, TO92-EBC, symbol BC237
Connections:
- net labels added: erreur_1, erreur_2, erreur_3, temoin_cmd+
- wire segments 169 -> 189
- no-connect marks 5 -> 19
Other:
- note added: "Erreurs Analog IN"
- note added: "MEZZA"
- note added: "Temoin CMD+"
- note added: "Temoins erreurs"

Commit message: 
Parts:
- C2, C4, C6, C8: value 100u -> 1u
Connections:
- wire segments 189 -> 194

Commit message: 
Parts:
- C1, C3, C5, C7: value 100n -> 27p
- P1: value clign -> clign_in
- P10: value codes -> codes_out
- P11: value pleins_feux -> pleins_feux_out
- P12: value commutateur 6pos -> commutateur_6_pos_in
- P13: value erreur_analog -> erreur_analog_in
- P14: value erreur_1 -> erreur_1_out
- P15: value erreur_2 -> erreur_2_out
- P16: value erreur_3 -> erreur_3_out
- P17: value cmd+ -> cmd+_out
- P2: value warning -> warning_in
- P3: value brake_analog -> brake_analog_out
- P4: value brake_input -> brake_in
- P5: value boost_analog -> boost_analog_out
- P6: value boost_input -> boost_in
- P7: value clign_g -> clign_g_out
- P8: value clign_d -> clign_d_out
Changed lines of the file:
@@
-EESchema Schematic File Version 2  date 07/04/2011 13:21:05
+EESchema Schematic File Version 2  date 07/04/2011 16:33:17
 LIBS:symbioz
 LIBS:epsa_relais
@@
 LIBS:contrib
 LIBS:valves
-LIBS:carte_tdb_v0.1-cache
-EELAYER 24  0
+EELAYER 25  0
 EELAYER END
 $Descr A4 11700 8267
+encoding utf-8
 Sheet 1 1
 Title "noname.sch"
@@
 P 10950 2600
 F 0 "P17" V 10900 2600 40  0000 C CNN
-F 1 "cmd+" V 11000 2600 40  0000 C CNN
+F 1 "cmd+_out" V 11000 2600 40  0000 C CNN
 	1    10950 2600
 	1    0    0    -1
@@
 P 10900 800
 F 0 "P16" V 10850 800 40  0000 C CNN
-F 1 "erreur_3" V 10950 800 40  0000 C CNN
+F 1 "erreur_3_out" V 10950 800 40  0000 C CNN
 	1    10900 800
 	1    0    0    -1
@@
 P 8900 800
 F 0 "P14" V 8850 800 40  0000 C CNN
-F 1 "erreur_1" V 8950 800 40  0000 C CNN
+F 1 "erreur_1_out" V 8950 800 40  0000 C CNN
 	1    8900 800
 	1    0    0    -1
@@
 P 8900 1400
 F 0 "P15" V 8850 1400 40  0000 C CNN
-F 1 "erreur_2" V 8950 1400 40  0000 C CNN
+F 1 "erreur_2_out" V 8950 1400 40  0000 C CNN
 	1    8900 1400
 	1    0    0    -1
@@
 P 5900 1050
 F 0 "P13" V 5850 1050 40  0000 C CNN
-F 1 "erreur_analog" V 5950 1050 40  0000 C CNN
+F 1 "erreur_analog_in" V 5950 1050 40  0000 C CNN
 	1    5900 1050
 	-1   0    0    1
@@
 P 3400 2500
 F 0 "C3" H 3300 2600 50  0000 L CNN
-F 1 "100n" H 3300 2400 50  0000 L CNN
+F 1 "27p" H 3300 2400 50  0000 L CNN
 	1    3400 2500
 	0    1    1    0
@@
 P 7900 3400
 F 0 "C7" H 7800 3500 50  0000 L CNN
-F 1 "100n" H 7800 3300 50  0000 L CNN
+F 1 "27p" H 7800 3300 50  0000 L CNN
 	1    7900 3400
 	0    1    1    0
@@
 P 6650 3400
 F 0 "C5" H 6550 3500 50  0000 L CNN
-F 1 "100n" H 6550 3300 50  0000 L CNN
+F 1 "27p" H 6550 3300 50  0000 L CNN
 	1    6650 3400
 	0    1    1    0
@@
 P 4250 3000
 F 0 "P12" V 4200 3000 60  0000 C CNN
-F 1 "commutateur 6pos" V 4300 3000 60  0000 C CNN
+F 1 "commutateur_6_pos_in" V 4300 3000 60  0000 C CNN
 	1    4250 3000
 	-1   0    0    1
@@
 P 6250 6800
 F 0 "P11" V 6200 6800 40  0000 C CNN
-F 1 "pleins_feux" V 6300 6800 40  0000 C CNN
+F 1 "pleins_feux_out" V 6300 6800 40  0000 C CNN
 	1    6250 6800
 	1    0    0    -1
@@
 P 6250 6200
 F 0 "P10" V 6200 6200 40  0000 C CNN
-F 1 "codes" V 6300 6200 40  0000 C CNN
+F 1 "codes_out" V 6300 6200 40  0000 C CNN
 	1    6250 6200
 	1    0    0    -1
@@
 P 5700 4450
 F 0 "C1" H 5600 4550 50  0000 L CNN
-F 1 "100n" H 5600 4350 50  0000 L CNN
+F 1 "27p" H 5600 4350 50  0000 L CNN
 	1    5700 4450
 	0    1    1    0
@@
 P 4300 6350
 F 0 "P7" V 4250 6350 40  0000 C CNN
-F 1 "clign_g" V 4350 6350 40  0000 C CNN
+F 1 "clign_g_out" V 4350 6350 40  0000 C CNN
 	1    4300 6350
 	1    0    0    -1
@@
 P 4300 6950
 F 0 "P8" V 4250 6950 40  0000 C CNN
-F 1 "clign_d" V 4350 6950 40  0000 C CNN
+F 1 "clign_d_out" V 4350 6950 40  0000 C CNN
 	1    4300 6950
 	1    0    0    -1
@@
 P 1000 7100
 F 0 "P2" V 950 7100 40  0000 C CNN
-F 1 "warning" V 1050 7100 40  0000 C CNN
+F 1 "warning_in" V 1050 7100 40  0000 C CNN
 	1    1000 7100
 	-1   0    0    1
@@
 P 1000 6400
 F 0 "P1" V 950 6400 50  0000 C CNN
-F 1 "clign" V 1050 6400 50  0000 C CNN
+F 1 "clign_in" V 1050 6400 50  0000 C CNN
 	1    1000 6400
 	-1   0    0    1
@@
 P 1050 4750
 F 0 "P5" V 1000 4750 40  0000 C CNN
-F 1 "boost_analog" V 1100 4750 40  0000 C CNN
+F 1 "boost_analog_out" V 1100 4750 40  0000 C CNN
 	1    1050 4750
 	-1   0    0    -1
@@
 P 1050 5200
 F 0 "P6" V 1000 5200 40  0000 C CNN
-F 1 "boost_input" V 1100 5200 40  0000 C CNN
+F 1 "boost_in" V 1100 5200 40  0000 C CNN
 	1    1050 5200
 	-1   0    0    -1
@@
 P 1050 3400
 F 0 "P4" V 1000 3400 40  0000 C CNN
-F 1 "brake_input" V 1100 3400 40  0000 C CNN
+F 1 "brake_in" V 1100 3400 40  0000 C CNN
 	1    1050 3400
 	-1   0    0    -1
@@
 P 1050 2950
 F 0 "P3" V 1000 2950 40  0000 C CNN
-F 1 "brake_analog" V 1100 2950 40  0000 C CNN
+F 1 "brake_analog_out" V 1100 2950 40  0000 C CNN
 	1    1050 2950
 	-1   0    0    -1

Commit message: 
Parts:
- removed C7: 27p, symbol C
- removed C8: 1u, symbol CP
- removed U4: 4049, symbol 4049
- added P18, P19, P20, P21: CONN_1, symbol CONN_1
Connections:
- wire segments 194 -> 185
- no-connect marks 19 -> 23
Other:
- note added: "Trous mécaniques"

Commit message: 
Connections:
- wire segments 185 -> 184
