File: KiCad/2012_HypnoZ/carte_tdb_v0.1/carte_tdb_v0.1.sch (KiCad schematic (older format))
At the start: 53 parts, among them P1 clign_in, P10 codes_out, P11 pleins_feux_out, P12 commutateur_6_pos_in, P13 erreur_analog_in, P14 erreur_1_out, P15 erreur_2_out, P16 erreur_3_out, P17 cmd+_out, P18 CONN_1, P19 CONN_1, P2 warning_in, P20 CONN_1, P21 CONN_1, P3 brake_analog_out, P4 brake_in, P5 boost_analog_out, P6 boost_in, P7 clign_g_out, P8 clign_d_out, P9 feux_in, Q1 BC237, Q2 BC237, Q3 BC237, Q4 BC237, Q5 BC237, Q6 BC237, Q7 BC237, Q8 BC237, U1 TL082, U2 4071, U3 74LS348

Commit message: 
Parts:
- removed C3: 27p, symbol C
- removed C4: 1u, symbol CP
- removed R5: 10k, symbol R
- removed U1: TL082, symbol TL082
- added C? (x3): 27p, symbol C
- added C? (x2): 0.01u, symbol CP
- added C?: 1u, symbol CP
- added R?: 10k, symbol R
- added R?: 22k, symbol R
- added R?: 51k, symbol R
- added U?: LM555N, symbol LM555N
Connections:
- net labels added: horloge
- wire segments 184 -> 192
Other:
- note added: "Timer"

Commit message: 
Parts:
- removed C?: 0.01u, symbol CP
- removed P13: erreur_analog_in, symbol CONN_2
- removed P8: clign_d_out, symbol CONN_2
- removed Q1, Q2, Q3, Q4, Q5, Q6, Q7, Q8: BC237, TO92-EBC, symbol BC237
- added C3: 27p, symbol C
- added C4: 1u, symbol CP
- added C7: 10n, symbol C
- added P4: clign_d_out, symbol CONN_2
- added P6: erreur_analog_in, symbol CONN_4
- added Q1, Q2, Q3, Q4, Q5, Q6, Q7, Q8: MOSFET_N, symbol MOSFET_N
- added U2: 4071, symbol 4071
- C12: renamed from C?; value 0.01u -> 10u
- P16: renamed from P18; value CONN_1 -> MECA_1
- P17: renamed from P19; value CONN_1 -> MECA_2
- P18: renamed from P20; value CONN_1 -> MECA_3
- P19: renamed from P21; value CONN_1 -> MECA_4
- R14: renamed from R?; value 51k -> 72k
- R15: renamed from R?; value 22k -> 31k
- gave numbers to parts that had none: 6
- renumbered C5 to C8, C6 to C9, P6 to P10, P10 to P11, P11 to P12, P12 to P13, P17 to P20, P16 to P21, P7 to P3, P9 to P5, P3 to P7, P4 to P8, P5 to P9, R6 to R4, R7 to R5, R4 to R6, U2 to U1
Connections:
- net labels added: clk, err_1_analog, err_1_can, err_2_analog, err_2_can, err_3_analog, err_3_can
- net labels removed: horloge
- wire segments 192 -> 212
- no-connect marks 23 -> 21
Other:
- note added: "Logique clignos"
- note added: "Logique erreurs"
- note removed: "Logique"
- moved on the sheet: P10, P11, P12, P20, P3, P7, P8, P9

Commit message: 
Parts:
- added C13, C15: 27p, symbol C
- added C14: 100u, symbol CP
- added C16: 10u, symbol CP
- added U5: 7806, symbol 7805
Connections:
- net labels added: +6V
- wire segments 212 -> 226
Other:
- moved on the sheet: P10, P11, P12, P9

Commit message: Rempalcement clignoteur 555 Corrections mineurs .brd
Parts:
- removed U4: LM555N, symbol LM555N
- added P22: T_Alim, symbol CONN_2
- added U4: LM555CN, symbol LM555CN
Connections:
- wire segments 226 -> 227
Other:
- note added: "Trous mÃ©caniques"
- note added: "Témoin alim général"
- note removed: "Trous mécaniques"

Commit message: 
Parts:
- removed P17: MECA_2, symbol CONN_1
- removed P18: MECA_3, symbol CONN_1
- removed P19: MECA_4, symbol CONN_1
- added MECA2, MECA3, MECA4: MECA, symbol CONN_1
- MECA1: renamed from P16; value MECA_1 -> MECA
Changed lines of the file:
@@
-EESchema Schematic File Version 2  date 18/04/2011 14:31:55
+EESchema Schematic File Version 2  date 18/04/2011 15:07:34
 LIBS:power
 LIBS:device
@@
 Comment4 ""
 $EndDescr
+$Comp
+L CONN_1 MECA3
+U 1 1 4DAC3780
+P 10100 6850
+F 0 "MECA3" H 10180 6850 40  0000 L CNN
+F 1 "MECA" H 10100 6905 30  0001 C CNN
+	1    10100 6850
+	1    0    0    -1
+$EndComp
+NoConn ~ 9950 6850
+NoConn ~ 9950 6950
+$Comp
+L CONN_1 MECA4
+U 1 1 4DAC377F
+P 10100 6950
+F 0 "MECA4" H 10180 6950 40  0000 L CNN
+F 1 "MECA" H 10100 7005 30  0001 C CNN
+	1    10100 6950
+	1    0    0    -1
+$EndComp
+$Comp
+L CONN_1 MECA2
+U 1 1 4DAC3778
+P 10100 6750
+F 0 "MECA2" H 10180 6750 40  0000 L CNN
+F 1 "MECA" H 10100 6805 30  0001 C CNN
+	1    10100 6750
+	1    0    0    -1
+$EndComp
+NoConn ~ 9950 6750
 Connection ~ 9550 4650
 Wire Wire Line
@@
 	10250 5500 10800 5500
 Wire Wire Line
-	10800 4450 10800 5500
+	10800 5500 10800 4450
 Connection ~ 10100 4650
 Wire Wire Line
@@
 	7600 3150 7500 3150
 Wire Wire Line
-	7650 2900 7800 2900
+	7800 2900 7650 2900
 Wire Wire Line
 	7500 2950 7650 2950
 Wire Wire Line
-	7550 2500 7800 2500
+	7800 2500 7550 2500
 Wire Wire Line
 	7550 2500 7550 2750
@@
 	7100 5100 7100 5150
 Wire Wire Line
-	7450 5350 6850 5350
-Wire Wire Line
-	7450 4900 7450 5350
-Wire Wire Line
-	6850 4900 7450 4900
+	6850 5350 7450 5350
+Wire Wire Line
+	7450 5350 7450 4900
+Wire Wire Line
+	7450 4900 6850 4900
 Wire Wire Line
 	7100 4750 7000 4750
@@
 	4950 3900 600  3900
 Wire Wire Line
-	7500 2300 7800 2300
-Wire Wire Line
-	7500 2650 7500 2300
-Wire Wire Line
-	7600 2850 7500 2850
+	7800 2300 7500 2300
+Wire Wire Line
+	7500 2300 7500 2650
+Wire Wire Line
+	7500 2850 7600 2850
 Wire Wire Line
 	7600 2850 7600 2700
@@
 	7500 3050 7650 3050
 Wire Wire Line
-	7650 3100 7650 3050
-Wire Wire Line
-	7800 3100 7650 3100
+	7650 3050 7650 3100
+Wire Wire Line
+	7650 3100 7800 3100
 Wire Wire Line
 	7500 3250 7550 3250
@@
 Connection ~ 7050 6250
 Wire Wire Line
-	7050 6100 7050 6250
+	7050 6250 7050 6100
 Wire Wire Line
 	7050 6100 7150 6100
 Wire Wire Line
-	7500 6250 6900 6250
+	6900 6250 7500 6250
 Wire Wire Line
 	7500 6250 7500 6700
@@
 NoConn ~ 1350 1400
 NoConn ~ 5200 6300
-NoConn ~ 9950 6950
-NoConn ~ 9950 6850
-NoConn ~ 9950 6750
 NoConn ~ 9950 6650
 Text Notes 9700 6550 0    60   ~ 0
 Trous mÃ©caniques
 $Comp
-L CONN_1 P19
-U 1 1 4D9DCBFD
-P 10100 6950
-F 0 "P19" H 10180 6950 40  0000 L CNN
-F 1 "MECA_4" H 10100 7005 30  0001 C CNN
-	1    10100 6950
-	1    0    0    -1
-$EndComp
-$Comp
-L CONN_1 P18
-U 1 1 4D9DCBFC
-P 10100 6850
-F 0 "P18" H 10180 6850 40  0000 L CNN
-F 1 "MECA_3" H 10100 6905 30  0001 C CNN
-	1    10100 6850
-	1    0    0    -1
-$EndComp
-$Comp
-L CONN_1 P17
-U 1 1 4D9DCBFA
-P 10100 6750
-F 0 "P17" H 10180 6750 40  0000 L CNN
-F 1 "MECA_2" H 10100 6805 30  0001 C CNN
-	1    10100 6750
-	1    0    0    -1
-$EndComp
-$Comp
-L CONN_1 P16
+L CONN_1 MECA1
 U 1 1 4D9DCBF7
 P 10100 6650
-F 0 "P16" H 10180 6650 40  0000 L CNN
-F 1 "MECA_1" H 10100 6705 30  0001 C CNN
+F 0 "MECA1" H 10180 6650 40  0000 L CNN
+F 1 "MECA" H 10100 6705 30  0001 C CNN
 	1    10100 6650
 	1    0    0    -1
